File: HG_Breakout/HG_Breakout.sch (KiCad schematic (older format))
At the start: 23 parts, among them J1 USB_B_Micro, J2 Conn_02x10_Odd_Even, J3 Conn_01x25_Female, SW1 SW_Push, U1 MIC5219-3.3, U2 efm32hg310f64g-b-qfn32, X1 S2B-PH-SM4-TB(LF)(SN)

Commit message: Should be finished - take a look!
Parts:
- removed J1: USB_B_Micro, symbol Connector:USB_B_Micro
- added P1: 10118193-0001LF, 10118193-0001LF:FCI_10118193-0001LF, symbol 10118193-0001LF:10118193-0001LF
- C1, C10, C11, C12, C13, C2, C3, C4, C5, C6, C7, C8, C9: footprint (none) -> Capacitor_SMD:C_0805_2012Metric_Pad1.15x1.40mm_HandSolder
- D1: footprint (none) -> LED_SMD:LED_0805_2012Metric_Pad1.15x1.40mm_HandSolder
- J2: footprint (none) -> Connector_PinHeader_2.54mm:PinHeader_2x10_P2.54mm_Vertical
- J3: footprint (none) -> Connector_PinHeader_2.54mm:PinHeader_1x25_P2.54mm_Vertical
- R1, TH1: footprint (none) -> Resistor_SMD:R_0805_2012Metric_Pad1.15x1.40mm_HandSolder
- SW1: footprint (none) -> PTS645SK50SMTR92LFS:SW_PTS645SK50SMTR92LFS
- U1: footprint Package_TO_SOT_SMD:SOT-23-5 -> SOT95P280X145-5N:SOT95P280X145-5N
- U2: footprint (none) -> EFM32HG310F64G-A-QFN32:SL_EFM32G200F64-QFN32T
- X1: footprint S2B-PH-SM4-TB(LF)(SN) -> S2B-PH-SM4-TB_LF__SN_:S2B-PH-SM4-TB(LF)(SN)
Connections:
- wire segments 128 -> 125
- no-connect marks 13 -> 12
